Commit message: changed the rotatiolimits for joint 5 and 4 (I might need to recheck the arm lenghts and rotation limits to the irl)

File: ws_MARA/src/arm_description/urdf/ASSY.xacro (robot description, xacro)
@@ -122,5 +122,5 @@
     <child link="5th_link_1"/>
     <axis xyz="0.0 1.0 0.0"/>
-    <limit lower="-3.14159" upper="3.14159" effort="50.0" velocity="3.14"/>
+    <limit lower="-1.5708" upper="1.5708" effort="50.0" velocity="3.14"/>
     <dynamics damping="0.5" friction="0.3"/>
   </joint>
@@ -152,5 +152,5 @@
     <child link="end_effector_link"/>
     <axis xyz="0.0 0.0 1.0"/>
-    <limit lower="-1.5708" upper="1.5708" effort="30.0" velocity="3.14"/>
+    <limit lower="-3.14159" upper="3.14159" effort="30.0" velocity="3.14"/>
     <dynamics damping="0.5" friction="0.3"/>
   </joint>

File: ws_MARA/src/arm_description/urdf/arm.urdf.xacro (robot description, xacro)
@@ -122,5 +122,5 @@
     <child link="5th_link_1"/>
     <axis xyz="0.0 1.0 0.0"/>
-    <limit lower="-3.14159" upper="3.14159" effort="50.0" velocity="3.14"/>
+    <limit lower="-1.5708" upper="1.5708" effort="50.0" velocity="3.14"/>
     <dynamics damping="0.5" friction="0.3"/>
   </joint>
@@ -152,5 +152,5 @@
     <child link="end_effector_link"/>
     <axis xyz="0.0 0.0 1.0"/>
-    <limit lower="-1.5708" upper="1.5708" effort="30.0" velocity="3.14"/>
+    <limit lower="-3.14159" upper="3.14159" effort="30.0" velocity="3.14"/>
     <dynamics damping="0.5" friction="0.3"/>
   </joint>

File: ws_MARA/src/arm_description/urdf/ros2_control.xacro (robot description, xacro)
@@ -38,4 +38,14 @@
     <joint name="joint_4">
       <command_interface name="position">
+        <param name="min">-1.5708</param>
+        <param name="max">1.5708</param>
+      </command_interface>
+      <state_interface name="position">
+        <param name="initial_value">0.0</param>
+      </state_interface>
+      <state_interface name="velocity"/>
+    </joint>
+    <joint name="joint_5">
+      <command_interface name="position">
         <param name="min">-3.14159</param>
         <param name="max">3.14159</param>
@@ -46,14 +56,4 @@
       <state_interface name="velocity"/>
     </joint>
-    <joint name="joint_5">
-      <command_interface name="position">
-        <param name="min">-1.5708</param>
-        <param name="max">1.5708</param>
-      </command_interface>
-      <state_interface name="position">
-        <param name="initial_value">0.0</param>
-      </state_interface>
-      <state_interface name="velocity"/>
-    </joint>
   </ros2_control>
 </robot>

Commit message: added find file function to make gazebo.launch.py find the stl and generate visuals

File: ws_MARA/src/arm_description/urdf/ASSY.xacro (robot description, xacro)
@@ -15,5 +15,5 @@
       <origin xyz="0 0 0" rpy="0 0 0"/>
       <geometry>
-        <mesh filename="package://arm_description/meshes/base_link.stl" scale="0.001 0.001 0.001"/>
+        <mesh filename="file://$(find arm_description)/meshes/base_link.stl" scale="0.001 0.001 0.001"/>
       </geometry>
       <material name="silver"/>
@@ -22,5 +22,5 @@
       <origin xyz="0 0 0" rpy="0 0 0"/>
       <geometry>
-        <mesh filename="package://arm_description/meshes/base_link.stl" scale="0.001 0.001 0.001"/>
+        <mesh filename="file://$(find arm_description)/meshes/base_link.stl" scale="0.001 0.001 0.001"/>
       </geometry>
     </collision>
@@ -45,5 +45,5 @@
       <origin xyz="0 0 0" rpy="0 0 0"/>
       <geometry>
-        <mesh filename="package://arm_description/meshes/2nd_link_1.stl" scale="0.001 0.001 0.001"/>
+        <mesh filename="file://$(find arm_description)/meshes/2nd_link_1.stl" scale="0.001 0.001 0.001"/>
       </geometry>
       <material name="silver"/>
@@ -52,5 +52,5 @@
       <origin xyz="0 0 0" rpy="0 0 0"/>
       <geometry>
-        <mesh filename="package://arm_description/meshes/2nd_link_1.stl" scale="0.001 0.001 0.001"/>
+        <mesh filename="file://$(find arm_description)/meshes/2nd_link_1.stl" scale="0.001 0.001 0.001"/>
       </geometry>
     </collision>
@@ -75,5 +75,5 @@
       <origin xyz="0 0 0" rpy="0 0 0"/>
       <geometry>
-        <mesh filename="package://arm_description/meshes/3rd_link_1.stl" scale="0.001 0.001 0.001"/>
+        <mesh filename="file://$(find arm_description)/meshes/3rd_link_1.stl" scale="0.001 0.001 0.001"/>
       </geometry>
       <material name="silver"/>
@@ -82,5 +82,5 @@
       <origin xyz="0 0 0" rpy="0 0 0"/>
       <geometry>
-        <mesh filename="package://arm_description/meshes/3rd_link_1.stl" scale="0.001 0.001 0.001"/>
+        <mesh filename="file://$(find arm_description)/meshes/3rd_link_1.stl" scale="0.001 0.001 0.001"/>
       </geometry>
     </collision>
@@ -105,5 +105,5 @@
       <origin xyz="0 0 0" rpy="0 0 0"/>
       <geometry>
-        <mesh filename="package://arm_description/meshes/4th_link_1.stl" scale="0.001 0.001 0.001"/>
+        <mesh filename="file://$(find arm_description)/meshes/4th_link_1.stl" scale="0.001 0.001 0.001"/>
       </geometry>
       <material name="silver"/>
@@ -112,5 +112,5 @@
       <origin xyz="0 0 0" rpy="0 0 0"/>
       <geometry>
-        <mesh filename="package://arm_description/meshes/4th_link_1.stl" scale="0.001 0.001 0.001"/>
+        <mesh filename="file://$(find arm_description)/meshes/4th_link_1.stl" scale="0.001 0.001 0.001"/>
       </geometry>
     </collision>
@@ -135,5 +135,5 @@
       <origin xyz="0 0 0" rpy="0 0 0"/>
       <geometry>
-        <mesh filename="package://arm_description/meshes/5th_link_1.stl" scale="0.001 0.001 0.001"/>
+        <mesh filename="file://$(find arm_description)/meshes/5th_link_1.stl" scale="0.001 0.001 0.001"/>
       </geometry>
       <material name="silver"/>
@@ -142,5 +142,5 @@
       <origin xyz="0 0 0" rpy="0 0 0"/>
       <geometry>
-        <mesh filename="package://arm_description/meshes/5th_link_1.stl" scale="0.001 0.001 0.001"/>
+        <mesh filename="file://$(find arm_description)/meshes/5th_link_1.stl" scale="0.001 0.001 0.001"/>
       </geometry>
     </collision>

File: ws_MARA/src/arm_description/urdf/arm.urdf.xacro (robot description, xacro)
@@ -15,5 +15,5 @@
       <origin xyz="0 0 0" rpy="0 0 0"/>
       <geometry>
-        <mesh filename="package://arm_description/meshes/base_link.stl" scale="0.001 0.001 0.001"/>
+        <mesh filename="file://$(find arm_description)/meshes/base_link.stl" scale="0.001 0.001 0.001"/>
       </geometry>
       <material name="silver"/>
@@ -22,5 +22,5 @@
       <origin xyz="0 0 0" rpy="0 0 0"/>
       <geometry>
-        <mesh filename="package://arm_description/meshes/base_link.stl" scale="0.001 0.001 0.001"/>
+        <mesh filename="file://$(find arm_description)/meshes/base_link.stl" scale="0.001 0.001 0.001"/>
       </geometry>
     </collision>
@@ -45,5 +45,5 @@
       <origin xyz="0 0 0" rpy="0 0 0"/>
       <geometry>
-        <mesh filename="package://arm_description/meshes/2nd_link_1.stl" scale="0.001 0.001 0.001"/>
+        <mesh filename="file://$(find arm_description)/meshes/2nd_link_1.stl" scale="0.001 0.001 0.001"/>
       </geometry>
       <material name="silver"/>
@@ -52,5 +52,5 @@
       <origin xyz="0 0 0" rpy="0 0 0"/>
       <geometry>
-        <mesh filename="package://arm_description/meshes/2nd_link_1.stl" scale="0.001 0.001 0.001"/>
+        <mesh filename="file://$(find arm_description)/meshes/2nd_link_1.stl" scale="0.001 0.001 0.001"/>
       </geometry>
     </collision>
@@ -75,5 +75,5 @@
       <origin xyz="0 0 0" rpy="0 0 0"/>
       <geometry>
-        <mesh filename="package://arm_description/meshes/3rd_link_1.stl" scale="0.001 0.001 0.001"/>
+        <mesh filename="file://$(find arm_description)/meshes/3rd_link_1.stl" scale="0.001 0.001 0.001"/>
       </geometry>
       <material name="silver"/>
@@ -82,5 +82,5 @@
       <origin xyz="0 0 0" rpy="0 0 0"/>
       <geometry>
-        <mesh filename="package://arm_description/meshes/3rd_link_1.stl" scale="0.001 0.001 0.001"/>
+        <mesh filename="file://$(find arm_description)/meshes/3rd_link_1.stl" scale="0.001 0.001 0.001"/>
       </geometry>
     </collision>
@@ -105,5 +105,5 @@
       <origin xyz="0 0 0" rpy="0 0 0"/>
       <geometry>
-        <mesh filename="package://arm_description/meshes/4th_link_1.stl" scale="0.001 0.001 0.001"/>
+        <mesh filename="file://$(find arm_description)/meshes/4th_link_1.stl" scale="0.001 0.001 0.001"/>
       </geometry>
       <material name="silver"/>
@@ -112,5 +112,5 @@
       <origin xyz="0 0 0" rpy="0 0 0"/>
       <geometry>
-        <mesh filename="package://arm_description/meshes/4th_link_1.stl" scale="0.001 0.001 0.001"/>
+        <mesh filename="file://$(find arm_description)/meshes/4th_link_1.stl" scale="0.001 0.001 0.001"/>
       </geometry>
     </collision>
@@ -135,5 +135,5 @@
       <origin xyz="0 0 0" rpy="0 0 0"/>
       <geometry>
-        <mesh filename="package://arm_description/meshes/5th_link_1.stl" scale="0.001 0.001 0.001"/>
+        <mesh filename="file://$(find arm_description)/meshes/5th_link_1.stl" scale="0.001 0.001 0.001"/>
       </geometry>
       <material name="silver"/>
@@ -142,5 +142,5 @@
       <origin xyz="0 0 0" rpy="0 0 0"/>
       <geometry>
-        <mesh filename="package://arm_description/meshes/5th_link_1.stl" scale="0.001 0.001 0.001"/>
+        <mesh filename="file://$(find arm_description)/meshes/5th_link_1.stl" scale="0.001 0.001 0.001"/>
       </geometry>
     </collision>
