Commit message: improvement: combined two gripper teeth as one prismatic and switched the direction of Elbow joint from the fusion2urdf assembly urdf

File: ws_MARA/src/marav2ckptbest_description/urdf/assemblies/marav2ckptbest.urdf.xacro (robot description, xacro)
@@ -216,5 +216,5 @@
       <child link="${prefix}elbow_arm"/>
       <origin xyz="-0.045000 0.000000 0.366000" rpy="-1.570796 0.000000 1.570796"/>
-      <axis xyz="0.000000 0.000000 1.000000"/>
+      <axis xyz="0.000000 0.000000 -1.000000"/>
       <limit effort="100.0" velocity="1.00"/>
     </joint>
@@ -243,4 +243,5 @@
       <origin xyz="0.000000 0.125000 0.000000" rpy="-1.570796 -1.570796 0.000000"/>
       <axis xyz="1.000000 0.000000 0.000000"/>
+      <mimic joint="${prefix}Slider_10" multiplier="-1.000000"/>
       <limit lower="-0.040000" upper="0.000000" effort="100.0" velocity="1.00"/>
     </joint>
@@ -298,6 +299,6 @@
       </joint>
       <joint name="${prefix}Slider_11">
-        <command_interface name="position"/>
-        <command_interface name="velocity"/>
+        <param name="mimic">${prefix}Slider_10</param>
+        <param name="multiplier">-1.0</param>
         <state_interface name="position">
           <param name="initial_value">0.0</param>

Commit message: improvement: added step movements for the digital twin when using the velocity controller.

File: ws_MARA/src/marav2ckptbest_description/urdf/assemblies/marav2ckptbest.urdf.xacro (robot description, xacro)
@@ -193,17 +193,17 @@
     </link>
     <!-- Joints (internal to assembly) -->
-    <joint name="${prefix}Revolute_1" type="continuous">
+    <joint name="${prefix}Revolute_1" type="revolute">
       <parent link="${prefix}base_link"/>
       <child link="${prefix}shoulder_link"/>
       <origin xyz="0.000000 0.000000 0.166000" rpy="0.000000 0.000000 0.000000"/>
       <axis xyz="0.000000 0.000000 1.000000"/>
-      <limit effort="100.0" velocity="1.00"/>
-    </joint>
-    <joint name="${prefix}Revolute_5" type="continuous">
+      <limit lower="-1.570796" upper="1.570796" effort="100.0" velocity="1.00"/>
+    </joint>
+    <joint name="${prefix}Revolute_5" type="revolute">
       <parent link="${prefix}shoulder_link"/>
       <child link="${prefix}shoulder_arm"/>
       <origin xyz="0.050000 0.000000 0.060000" rpy="1.570796 0.000000 1.570796"/>
       <axis xyz="0.000000 0.000000 1.000000"/>
-      <limit effort="100.0" velocity="1.00"/>
+      <limit lower="-1.570796" upper="1.570796" effort="100.0" velocity="1.00"/>
     </joint>
     <joint name="${prefix}Rigid_6" type="fixed">
@@ -212,10 +212,10 @@
       <origin xyz="0.000000 -0.226000 -0.050000" rpy="-1.570796 -1.570796 0.000000"/>
     </joint>
-    <joint name="${prefix}Revolute_7" type="continuous">
+    <joint name="${prefix}Revolute_7" type="revolute">
       <parent link="${prefix}elbow_link"/>
       <child link="${prefix}elbow_arm"/>
       <origin xyz="-0.045000 0.000000 0.366000" rpy="-1.570796 0.000000 1.570796"/>
       <axis xyz="0.000000 0.000000 -1.000000"/>
-      <limit effort="100.0" velocity="1.00"/>
+      <limit lower="-1.570796" upper="1.570796" effort="100.0" velocity="1.00"/>
     </joint>
     <joint name="${prefix}Rigid_8" type="fixed">
@@ -224,10 +224,10 @@
       <origin xyz="0.000000 0.366000 -0.045000" rpy="1.570796 1.570796 0.000000"/>
     </joint>
-    <joint name="${prefix}Revolute_9" type="continuous">
+    <joint name="${prefix}Revolute_9" type="revolute">
       <parent link="${prefix}wrist_link"/>
       <child link="${prefix}wrist_arm"/>
       <origin xyz="0.050000 0.000000 0.506000" rpy="1.570796 0.000000 1.570796"/>
       <axis xyz="0.000000 0.000000 1.000000"/>
-      <limit effort="100.0" velocity="1.00"/>
+      <limit lower="-1.570796" upper="1.570796" effort="100.0" velocity="1.00"/>
     </joint>
     <joint name="${prefix}Slider_10" type="prismatic">
@@ -249,5 +249,5 @@
     <ros2_control name="${prefix}marav2ckptbest_system" type="system">
       <hardware>
-        <plugin>mock_components/GenericSystem</plugin>
+        <plugin>marav2ckptbest_hardware/StepHardware</plugin>
         <param name="cmd_topic">sim/marav2ckptbest_system/cmd</param>
         <param name="state_topic">sim/marav2ckptbest_system/state</param>

File: ws_MARA/src/marav2ckptbest_description/urdf/marav2ckptbest.urdf (robot description, URDF)
Before this commit: robot marav2ckptbest, 9 links, 8 joints
Joints:
- joint Revolute_1: limit effort=100.0 velocity=1.00 -> lower=-1.570796 upper=1.570796 effort=100.0 velocity=1.00; type continuous -> revolute
- joint Revolute_5: limit effort=100.0 velocity=1.00 -> lower=-1.570796 upper=1.570796 effort=100.0 velocity=1.00; type continuous -> revolute
- joint Revolute_7: limit effort=100.0 velocity=1.00 -> lower=-1.570796 upper=1.570796 effort=100.0 velocity=1.00; type continuous -> revolute
- joint Revolute_9: limit effort=100.0 velocity=1.00 -> lower=-1.570796 upper=1.570796 effort=100.0 velocity=1.00; type continuous -> revolute
