Commit message: feat: added the top and bottom cameras placed beside the end effector tool changer attachment as well as camera message simulation scripts

File: ws_MARA/src/marav3best_description/marav3best_description/urdf/assemblies/marav3best.urdf.xacro (robot description, xacro)
@@ -1,5 +1,5 @@
 <?xml version="1.0"?>
 <robot xmlns:xacro="http://www.ros.org/wiki/xacro" name="marav3best_macro">
-  <xacro:macro name="marav3best" params="prefix">
+  <xacro:macro name="marav3best" params="prefix use_sim:=false">
     <!-- Links -->
     <link name="${prefix}base_link">
@@ -333,11 +333,16 @@
       <mimic joint="${prefix}J9_horn_drive" multiplier="-1.0" offset="0.0"/>
     </joint>
-    <!-- ROS 2 control: generated generic system -->
+    <!-- ROS 2 control: mock hardware for RViz, gz_ros2_control for Gazebo -->
     <ros2_control name="${prefix}marav3best_system" type="system">
       <hardware>
-        <plugin>mock_components/GenericSystem</plugin>
-        <param name="cmd_topic">sim/marav3best_system/cmd</param>
-        <param name="state_topic">sim/marav3best_system/state</param>
-        <param name="calculate_dynamics">true</param>
+        <xacro:if value="${use_sim}">
+          <plugin>gz_ros2_control/GazeboSimSystem</plugin>
+        </xacro:if>
+        <xacro:unless value="${use_sim}">
+          <plugin>mock_components/GenericSystem</plugin>
+          <param name="cmd_topic">sim/marav3best_system/cmd</param>
+          <param name="state_topic">sim/marav3best_system/state</param>
+          <param name="calculate_dynamics">true</param>
+        </xacro:unless>
       </hardware>
       <joint name="${prefix}J1_yaw_base_shoulderLink">
@@ -386,4 +391,19 @@
         <state_interface name="effort"/>
       </joint>
+      <!-- Gripper linkage follows J9 through the URDF <mimic> tags; Gazebo
+           only drives mimic joints that are listed here -->
+      <xacro:if value="${use_sim}">
+        <xacro:macro name="mimic_state" params="name">
+          <joint name="${prefix}${name}">
+            <state_interface name="position"/>
+            <state_interface name="velocity"/>
+            <state_interface name="effort"/>
+          </joint>
+        </xacro:macro>
+        <xacro:mimic_state name="J10_horn_link1"/>
+        <xacro:mimic_state name="J11_horn_link2"/>
+        <xacro:mimic_state name="J12_link1_tooth1"/>
+        <xacro:mimic_state name="J13_link2_tooth2"/>
+      </xacro:if>
     </ros2_control>
   </xacro:macro>

File: ws_MARA/src/marav3best_description/marav3best_description/urdf/marav3best.urdf.xacro (robot description, xacro)
@@ -7,5 +7,23 @@
   <!-- Assembly includes -->
   <xacro:include filename="$(find marav3best_description)/urdf/assemblies/marav3best.urdf.xacro"/>
+  <xacro:include filename="$(find marav3best_description)/urdf/stereo_camera.urdf.xacro"/>
+  <!-- use_sim:=true swaps mock hardware for Gazebo (gz_ros2_control) -->
+  <xacro:arg name="use_sim" default="false"/>
+  <xacro:property name="use_sim" value="$(arg use_sim)"/>
   <!-- Instantiate assemblies -->
-  <xacro:marav3best prefix=""/>
+  <xacro:marav3best prefix="" use_sim="${use_sim}"/>
+  <xacro:stereo_pair prefix=""/>
+  <xacro:if value="${use_sim}">
+    <link name="world"/>
+    <joint name="world_to_base" type="fixed">
+      <parent link="world"/>
+      <child link="base_link"/>
+      <origin xyz="0 0 0" rpy="0 0 0"/>
+    </joint>
+    <gazebo>
+      <plugin filename="gz_ros2_control-system" name="gz_ros2_control::GazeboSimROS2ControlPlugin">
+        <parameters>$(find marav3best_description)/config/ros2_controllers.yaml</parameters>
+      </plugin>
+    </gazebo>
+  </xacro:if>
 </robot>
